File: SLAMP.sch (EAGLE design)
At the start: 57 parts, among them IC1 MEGA8-AI, IC2 AT42QT1070-SSU, J1 CARA1, J2 CARA4, J3 CARA2, J4 CARA5, J5 CARA3, J6 EXTRA-D12, J7 A0, Q1 2N7002PW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

Commit message: Atmega328p finished
Connections:
- net B_RX renamed D11/MOSI
- net D13 renamed D13/SCK
- removed net D12: ISP1.MISO, J6.1
- removed net N$22: IC1.ADC7
- removed net N$7: IC1.ADC6
- new net D10: IC1.PB2(SS/OC1B)
- new net D12/MISO: IC1.PB4(MISO), ISP1.MISO, J6.1
- net B_TX: no longer IC1.PB2(SS/OC1B)
- net SCL: now also IC1.PC5(ADC5/SCL)
- net SDA: now also IC1.PC4(ADC4/SDA)
Other:
- moved on the sheet: ISP1, LED1, LED2, R10, R8
Changed lines of the file:
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@@
 <wire x1="116.84" y1="114.3" x2="116.84" y2="190.5" width="0.1524" layer="150"/>
 <text x="119.38" y="116.84" size="2.54" layer="150">Bluetooth Connectivity</text>
+<wire x1="248.92" y1="-53.34" x2="276.86" y2="-53.34" width="0.1524" layer="150"/>
+<wire x1="276.86" y1="-53.34" x2="276.86" y2="-114.3" width="0.1524" layer="150"/>
+<wire x1="276.86" y1="-114.3" x2="248.92" y2="-114.3" width="0.1524" layer="150"/>
 </plain>
 <instances>
@@
 <instance part="SUPPLY18" gate="G$1" x="332.74" y="132.08"/>
 <instance part="SUPPLY19" gate="G$1" x="287.02" y="109.22"/>
-<instance part="ISP1" gate="G$1" x="236.22" y="-22.86"/>
-<instance part="GND28" gate="1" x="254" y="-30.48"/>
-<instance part="SUPPLY20" gate="G$1" x="254" y="-17.78"/>
+<instance part="ISP1" gate="G$1" x="566.42" y="177.8"/>
+<instance part="GND28" gate="1" x="584.2" y="170.18"/>
+<instance part="SUPPLY20" gate="G$1" x="584.2" y="182.88"/>
 <instance part="R7" gate="G$1" x="195.58" y="147.32"/>
-<instance part="LED1" gate="G$1" x="431.8" y="45.72" rot="R90"/>
-<instance part="LED2" gate="G$1" x="431.8" y="55.88" rot="R90"/>
-<instance part="R8" gate="G$1" x="419.1" y="45.72" rot="R180"/>
-<instance part="R10" gate="G$1" x="419.1" y="55.88" rot="R180"/>
+<instance part="LED1" gate="G$1" x="269.24" y="-76.2" rot="R180"/>
+<instance part="LED2" gate="G$1" x="259.08" y="-76.2" rot="R180"/>
+<instance part="R8" gate="G$1" x="269.24" y="-88.9" rot="R270"/>
+<instance part="R10" gate="G$1" x="259.08" y="-88.9" rot="R270"/>
 <instance part="GND16" gate="1" x="15.24" y="71.12"/>
 <instance part="GND17" gate="1" x="48.26" y="71.12"/>
@@
 <segment>
 <pinref part="ISP1" gate="G$1" pin="RST"/>
-<wire x1="223.52" y1="-25.4" x2="220.98" y2="-25.4" width="0.1524" layer="91"/>
-<label x="220.98" y="-25.4" size="1.016" layer="95" rot="R180" xref="yes"/>
+<wire x1="553.72" y1="175.26" x2="551.18" y2="175.26" width="0.1524" layer="91"/>
+<label x="551.18" y="175.26" size="1.016" layer="95" rot="R180" xref="yes"/>
 </segment>
 </net>
@@
 <pinref part="ISP1" gate="G$1" pin="GND"/>
 <pinref part="GND28" gate="1" pin="GND"/>
-<wire x1="251.46" y1="-25.4" x2="254" y2="-25.4" width="0.1524" layer="91"/>
-<wire x1="254" y1="-25.4" x2="254" y2="-27.94" width="0.1524" layer="91"/>
+<wire x1="581.66" y1="175.26" x2="584.2" y2="175.26" width="0.1524" layer="91"/>
+<wire x1="584.2" y1="175.26" x2="584.2" y2="172.72" width="0.1524" layer="91"/>
 </segment>
 <segment>
@@
 </segment>
 </net>
-<net name="D13" class="0">
+<net name="D13/SCK" class="0">
 <segment>
 <pinref part="IC1" gate="G$1" pin="PB5(SCK)"/>
@@
 <segment>
 <pinref part="ISP1" gate="G$1" pin="SCK"/>
-<wire x1="223.52" y1="-22.86" x2="220.98" y2="-22.86" width="0.1524" layer="91"/>
-<label x="220.98" y="-22.86" size="1.016" layer="95" rot="R180" xref="yes"/>
+<wire x1="553.72" y1="177.8" x2="551.18" y2="177.8" width="0.1524" layer="91"/>
+<label x="551.18" y="177.8" size="1.016" layer="95" rot="R180" xref="yes"/>
 </segment>
 </net>
@@
 <wire x1="289.56" y1="106.68" x2="284.48" y2="106.68" width="0.1524" layer="91"/>
 <label x="284.48" y="106.68" size="1.016" layer="95" rot="R180" xref="yes"/>
-</segment>
-</net>
-<net name="D12" class="0">
-<segment>
-<pinref part="J6" gate="G$1" pin="1"/>
-<wire x1="335.28" y1="129.54" x2="330.2" y2="129.54" width="0.1524" layer="91"/>
-<label x="330.2" y="129.54" size="1.016" layer="95" rot="R180" xref="yes"/>
-</segment>
-<segment>
-<pinref part="ISP1" gate="G$1" pin="MISO"/>
-<wire x1="223.52" y1="-20.32" x2="220.98" y2="-20.32" width="0.1524" layer="91"/>
-<label x="220.98" y="-20.32" size="1.016" layer="95" rot="R180" xref="yes"/>
 </segment>
 </net>
@@
 <pinref part="ISP1" gate="G$1" pin="VCC"/>
 <pinref part="SUPPLY20" gate="G$1" pin="5V"/>
-<wire x1="251.46" y1="-20.32" x2="254" y2="-20.32" width="0.1524" layer="91"/>
-<wire x1="254" y1="-20.32" x2="254" y2="-17.78" width="0.1524" layer="91"/>
+<wire x1="581.66" y1="180.34" x2="584.2" y2="180.34" width="0.1524" layer="91"/>
+<wire x1="584.2" y1="180.34" x2="584.2" y2="182.88" width="0.1524" layer="91"/>
 </segment>
 <segment>
@@
 <segment>
 <pinref part="LED2" gate="G$1" pin="C"/>
-<wire x1="436.88" y1="55.88" x2="441.96" y2="55.88" width="0.1524" layer="91"/>
-<label x="441.96" y="55.88" size="1.016" layer="95" xref="yes"/>
+<wire x1="259.08" y1="-71.12" x2="259.08" y2="-66.04" width="0.1524" layer="91"/>
+<label x="259.08" y="-66.04" size="1.016" layer="95" rot="R90" xref="yes"/>
 </segment>
 </net>
@@
 <segment>
 <pinref part="LED1" gate="G$1" pin="C"/>
-<wire x1="441.96" y1="45.72" x2="436.88" y2="45.72" width="0.1524" layer="91"/>
-<label x="441.96" y="45.72" size="1.016" layer="95" xref="yes"/>
+<wire x1="269.24" y1="-66.04" x2="269.24" y2="-71.12" width="0.1524" layer="91"/>
+<label x="269.24" y="-66.04" size="1.016" layer="95" rot="R90" xref="yes"/>
 </segment>
 </net>
@@
 <label x="127" y="172.72" size="1.27" layer="95" rot="R180" xref="yes"/>
 </segment>
-<segment>
-<pinref part="IC1" gate="G$1" pin="PB2(SS/OC1B)"/>
-<wire x1="518.16" y1="129.54" x2="528.32" y2="129.54" width="0.1524" layer="91"/>
-<label x="528.32" y="129.54" size="1.27" layer="95" xref="yes"/>
-</segment>
-</net>
-<net name="B_RX" class="0">
-<segment>
-<pinref part="U1" gate="G$1" pin="RX"/>
-<wire x1="139.7" y1="170.18" x2="127" y2="170.18" width="0.1524" layer="91"/>
-<label x="127" y="170.18" size="1.27" layer="95" rot="R180" xref="yes"/>
-</segment>
-<segment>
-<pinref part="IC1" gate="G$1" pin="PB3(MOSI/OC2)"/>
-<wire x1="518.16" y1="127" x2="528.32" y2="127" width="0.1524" layer="91"/>
-<label x="528.32" y="127" size="1.27" layer="95" xref="yes"/>
-</segment>
-<segment>
-<pinref part="ISP1" gate="G$1" pin="MOSI"/>
-<wire x1="251.46" y1="-22.86" x2="254" y2="-22.86" width="0.1524" layer="91"/>
-<label x="254" y="-22.86" size="1.016" layer="95" xref="yes"/>
-</segment>
 </net>
 <net name="KEY" class="0">
@@
 <pinref part="R8" gate="G$1" pin="1"/>
 <pinref part="LED1" gate="G$1" pin="A"/>
-<wire x1="424.18" y1="45.72" x2="429.26" y2="45.72" width="0.1524" layer="91"/>
+<wire x1="269.24" y1="-83.82" x2="269.24" y2="-78.74" width="0.1524" layer="91"/>
 </segment>
 </net>
@@
 <pinref part="R10" gate="G$1" pin="1"/>
 <pinref part="LED2" gate="G$1" pin="A"/>
-<wire x1="424.18" y1="55.88" x2="429.26" y2="55.88" width="0.1524" layer="91"/>
+<wire x1="259.08" y1="-83.82" x2="259.08" y2="-78.74" width="0.1524" layer="91"/>
 </segment>
 </net>
@@
 <segment>
 <pinref part="R10" gate="G$1" pin="2"/>
-<wire x1="411.48" y1="55.88" x2="414.02" y2="55.88" width="0.1524" layer="91"/>
-<label x="411.48" y="55.88" size="1.016" layer="95" rot="R180" xref="yes"/>
+<wire x1="259.08" y1="-96.52" x2="259.08" y2="-93.98" width="0.1524" layer="91"/>
+<label x="259.08" y="-96.52" size="1.016" layer="95" rot="R270" xref="yes"/>
 </segment>
 <segment>
 <pinref part="R8" gate="G$1" pin="2"/>
-<wire x1="411.48" y1="45.72" x2="414.02" y2="45.72" width="0.1524" layer="91"/>
-<label x="411.48" y="45.72" size="1.016" layer="95" rot="R180" xref="yes"/>
+<wire x1="269.24" y1="-96.52" x2="269.24" y2="-93.98" width="0.1524" layer="91"/>
+<label x="269.24" y="-96.52" size="1.016" layer="95" rot="R270" xref="yes"/>
 </segment>
 </net>
@@
 <junction x="396.24" y="-12.7"/>
 </segment>
+<segment>
+<pinref part="IC1" gate="G$1" pin="PC4(ADC4/SDA)"/>
+<wire x1="518.16" y1="170.18" x2="528.32" y2="170.18" width="0.1524" layer="91"/>
+<label x="528.32" y="170.18" size="1.016" layer="95" xref="yes"/>
+</segment>
 </net>
 <net name="SCL" class="0">
@@
 <junction x="401.32" y="-20.32"/>
 </segment>
+<segment>
+<pinref part="IC1" gate="G$1" pin="PC5(ADC5/SCL)"/>
+<wire x1="518.16" y1="167.64" x2="528.32" y2="167.64" width="0.1524" layer="91"/>
+<label x="528.32" y="167.64" size="1.016" layer="95" xref="yes"/>
+</segment>
 </net>
 <net name="N$30" class="0">
@@
 </segment>
 </net>
-<net name="N$7" class="0">
-<segment>
-<pinref part="IC1" gate="G$1" pin="ADC6"/>
-<wire x1="518.16" y1="165.1" x2="520.7" y2="165.1" width="0.1524" layer="91"/>
-</segment>
-</net>
-<net name="N$22" class="0">
-<segment>
-<pinref part="IC1" gate="G$1" pin="ADC7"/>
-<wire x1="518.16" y1="162.56" x2="520.7" y2="162.56" width="0.1524" layer="91"/>
-</segment>
-</net>
 <net name="BT_TX" class="0">
 <segment>
@@
 </segment>
 </net>
+<net name="D12/MISO" class="0">
+<segment>
+<pinref part="IC1" gate="G$1" pin="PB4(MISO)"/>
+<wire x1="518.16" y1="124.46" x2="528.32" y2="124.46" width="0.1524" layer="91"/>
+<label x="528.32" y="124.46" size="1.016" layer="95" xref="yes"/>
+</segment>
+<segment>
+<pinref part="J6" gate="G$1" pin="1"/>
+<wire x1="335.28" y1="129.54" x2="330.2" y2="129.54" width="0.1524" layer="91"/>
+<label x="330.2" y="129.54" size="1.016" layer="95" rot="R180" xref="yes"/>
+</segment>
+<segment>
+<pinref part="ISP1" gate="G$1" pin="MISO"/>
+<wire x1="553.72" y1="180.34" x2="551.18" y2="180.34" width="0.1524" layer="91"/>
+<label x="551.18" y="180.34" size="1.016" layer="95" rot="R180" xref="yes"/>
+</segment>
+</net>
+<net name="D11/MOSI" class="0">
+<segment>
+<pinref part="IC1" gate="G$1" pin="PB3(MOSI/OC2)"/>
+<wire x1="518.16" y1="127" x2="528.32" y2="127" width="0.1524" layer="91"/>
+<label x="528.32" y="127" size="1.016" layer="95" xref="yes"/>
+</segment>
+<segment>
+<pinref part="U1" gate="G$1" pin="RX"/>
+<wire x1="139.7" y1="170.18" x2="127" y2="170.18" width="0.1524" layer="91"/>
+<label x="127" y="170.18" size="1.27" layer="95" rot="R180" xref="yes"/>
+</segment>
+<segment>
+<pinref part="ISP1" gate="G$1" pin="MOSI"/>
+<wire x1="581.66" y1="177.8" x2="584.2" y2="177.8" width="0.1524" layer="91"/>
+<label x="584.2" y="177.8" size="1.016" layer="95" xref="yes"/>
+</segment>
+</net>
+<net name="D10" class="0">
+<segment>
+<pinref part="IC1" gate="G$1" pin="PB2(SS/OC1B)"/>
+<wire x1="518.16" y1="129.54" x2="528.32" y2="129.54" width="0.1524" layer="91"/>
+<label x="528.32" y="129.54" size="1.016" layer="95" xref="yes"/>
+</segment>
+</net>

Commit message: Improving schematic
Parts:
- added FRAME1: FRAME-LETTERNO_PACKAGE, SparkFun-Aesthetics:FRAME-LETTERNO_PACKAGE
- J6: value EXTRA-D12 -> EXTRA-D10
Connections:
- removed net B_TX: U1.TX
- removed net D11/MOSI: IC1.PB3(MOSI/OC2), ISP1.MOSI, U1.RX
- removed net D12/MISO: IC1.PB4(MISO), ISP1.MISO, J6.1
- removed net D2: J1.1
- removed net D3: J3.1
- removed net D4: IC1.PD4(XCK/T0), J5.1
- removed net D5: IC1.PD5(T1), J2.1
- removed net D6: IC1.PD6(AIN0), J4.1
- net BT_RX: now also ISP1.MOSI, U1.RX
- net BT_TX: now also U1.TX
- net D10: now also IC1.PB4(MISO), ISP1.MISO, J6.1
- net D7: now also IC1.PD5(T1), J2.1, J3.1
- net D8: now also IC1.PD4(XCK/T0), IC1.PD6(AIN0), J1.1, J4.1, J5.1

Commit message: Changing schematic
Parts:
- removed C1, C3: 100n, SparkFun-Passives:CAP0805
- removed C2, C5: 0.1u, SparkFun-Passives:CAP0603-CAP
- removed C4: 0.1u, SparkFun-Passives:CAP0805
- removed C6: 10u, rcl:CPOL-USSMCP
- removed D2: GREEN, SparkFun-LED:LED-BLUE0603
- removed IC1: MEGA8-AI, atmel:MEGA8-AI
- removed R2: 10k, SparkFun-Passives:RESISTOR0805-RES
- removed R3: 1k, SparkFun-Passives:RESISTOR0805-RES
- removed S1: SWITCH-MOMENTARY-2PTH, SparkFun-Electromechanical:SWITCH-MOMENTARY-2PTH
- removed Y1: 16MHZ, SparkFun-FreqCtrl:RESONATOR16MHZ
- added C16, C7: 100n, SparkFun-Passives:CAP0805
- added C17: 0.1u, SparkFun-Passives:CAP0805
- added C18, C19: 0.1u, SparkFun-Passives:CAP0603-CAP
- added C20: 10u, rcl:CPOL-USSMCP
- added D3: GREEN, SparkFun-LED:LED-BLUE0603
- added FRAME2: FRAME-LETTERNO_PACKAGE, SparkFun-Aesthetics:FRAME-LETTERNO_PACKAGE
- added R1: 10k, SparkFun-Passives:RESISTOR0805-RES
- added R18: 1k, SparkFun-Passives:RESISTOR0805-RES
- added S2: SWITCH-MOMENTARY-2PTH, SparkFun-Electromechanical:SWITCH-MOMENTARY-2PTH
- added U2: MIC5219 3.3V, SparkFun-PowerIC:V_REG_MIC52193.3V
- added Y2: 16MHZ, SparkFun-FreqCtrl:RESONATOR16MHZ
- U3: value MIC5219 3.3V -> ATMEGA328P_TQFP; device SparkFun-PowerIC:V_REG_MIC52193.3V -> SparkFun-DigitalIC:ATMEGA328P_TQFP
Connections:
- removed net KEY: IC1.PB1(OC1A)
- removed net N$6: D2.A, R3.1
- new net 11/MOSI: ISP1.MOSI, U3.PB3(MOSI/OC2)
- new net 12/MISO: ISP1.MISO, U3.PB4(MISO)
- new net D4: U3.PD4(XCK/T0)
- new net D5: U3.PD5(T1)
- new net D6: U3.PD6(AIN0)
- new net N$24: D3.A, R18.1
- net 3.3V: now also C19.1, C20.+, U2.OUT; no longer C5.1, C6.+, U3.OUT
- net 5V: now also C17.2, C18.2, R1.2, U2.EN, U2.IN, U3.AVCC, U3.VCC@4, U3.VCC@6; no longer C2.2, C4.2, IC1.AVCC, IC1.VCC@1, IC1.VCC@2, R2.2, U3.EN, U3.IN
- net A0: now also U3.PC0(ADC0); no longer IC1.PC0(ADC0)
- net BT_RX: now also U3.PD3(INT1); no longer IC1.PD3(INT1), ISP1.MOSI
- net BT_TX: now also U3.PD2(INT0); no longer IC1.PD2(INT0)
- net D10: now also U3.PB2(SS/OC1B); no longer IC1.PB2(SS/OC1B), IC1.PB4(MISO), ISP1.MISO
- net D13/SCK: now also R18.2, U3.PB5(SCK); no longer IC1.PB5(SCK), R3.2
- net D7: now also U3.PD7(AIN1); no longer IC1.PD5(T1), IC1.PD7(AIN1)
- net D8: now also U3.PB0(ICP); no longer IC1.PB0(ICP), IC1.PD4(XCK/T0), IC1.PD6(AIN0)
- net DTR: now also C7.1; no longer C1.1
- net GND: now also C16.1, C17.1, C18.1, C19.2, C20.-, D3.C, S2.1, U2.GND, U3.AGND, U3.GND@3, U3.GND@5, Y2.2; no longer C2.1, C3.1, C4.1, C5.2, C6.-, D2.C, IC1.GND, IC1.GND@1, IC1.GND@2, S1.1, U3.GND, Y1.2
- net N$2: now also U3.PB6(XTAL1/TOSC1), Y2.1; no longer C3.2, IC1.AREF
- net N$3: now also U3.PB7(XTAL2/TOSC2), Y2.3; no longer IC1.PB6(XTAL1/TOSC1), Y1.1
- net N$4: now also C16.2, U3.AREF; no longer IC1.PB7(XTAL2/TOSC2), Y1.3
- net RESET: now also C7.2, R1.1, S2.2, U3.PC6(/RESET); no longer C1.2, IC1.PC6(/RESET), R2.1, S1.2
- net RX: now also U3.PD0(RXD); no longer IC1.PD0(RXD)
- net SCL: now also U3.PC5(ADC5/SCL); no longer IC1.PC5(ADC5/SCL)
- net SDA: now also U3.PC4(ADC4/SDA); no longer IC1.PC4(ADC4/SDA)
- net TX: now also U3.PD1(TXD); no longer IC1.PD1(TXD)
