File: SLAMP.brd (EAGLE design)
At the start: 160 x 100 mm, 57 parts, among them IC1 MEGA8-AI, IC2 AT42QT1070-SSU, J1 CARA1, J2 CARA4, J3 CARA2, J4 CARA5, J5 CARA3, J6 EXTRA-D12, J7 A0, Q1 2N7002PW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

Commit message: Atmega328p finished
Connections:
- net B_RX renamed D11/MOSI
- net D13 renamed D13/SCK
- removed net D12: ISP1.1, J6.1
- removed net N$22: IC1.22
- removed net N$7: IC1.19
- new net D10: IC1.14
- new net D12/MISO: IC1.16, ISP1.1, J6.1
- net B_TX: no longer IC1.14
- net SCL: now also IC1.28
- net SDA: now also IC1.27
Routing:
- net D12/MISO: track 0.00 -> 70.9 mm
- net D12: track 70.9 -> 0.00 mm
Changed lines of the file:
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@@
 <wire x1="42.2275" y1="75.4701" x2="42.285" y2="75.4126" width="0.254" layer="1"/>
 </signal>
-<signal name="D13">
+<signal name="D13/SCK">
 <contactref element="IC1" pad="17"/>
 <contactref element="R3" pad="2"/>
@@
 <wire x1="46.99" y1="69.215" x2="46.99" y2="66.9224" width="0.254" layer="1"/>
 <wire x1="46.99" y1="66.9224" x2="47.085" y2="66.8274" width="0.254" layer="1"/>
-</signal>
-<signal name="D12">
-<contactref element="J6" pad="1"/>
-<contactref element="ISP1" pad="1"/>
-<wire x1="47.9425" y1="68.2625" x2="47.9425" y2="70.1675" width="0.254" layer="1"/>
-<wire x1="47.9425" y1="70.1675" x2="47.625" y2="70.485" width="0.254" layer="1"/>
-<wire x1="47.625" y1="70.485" x2="45.72" y2="70.485" width="0.254" layer="1"/>
-<wire x1="45.72" y1="70.485" x2="45.085" y2="69.85" width="0.254" layer="1"/>
-<wire x1="45.085" y1="69.85" x2="45.085" y2="69.215" width="0.254" layer="1"/>
-<wire x1="45.085" y1="69.215" x2="44.1325" y2="68.2625" width="0.254" layer="1"/>
-<wire x1="44.1325" y1="68.2625" x2="40.8499" y2="68.2625" width="0.254" layer="1"/>
-<wire x1="47.9425" y1="68.2625" x2="48.895" y2="67.31" width="0.254" layer="1"/>
-<wire x1="48.895" y1="67.31" x2="51.435" y2="67.31" width="0.254" layer="1"/>
-<wire x1="51.435" y1="67.31" x2="51.435" y2="69.215" width="0.254" layer="1"/>
-<wire x1="51.435" y1="69.215" x2="52.705" y2="70.485" width="0.254" layer="1"/>
-<wire x1="52.705" y1="70.485" x2="54.6" y2="70.485" width="0.254" layer="1"/>
-<wire x1="54.6" y1="70.485" x2="54.695" y2="70.58" width="0.254" layer="1"/>
-<wire x1="17.78" y1="53.975" x2="33.655" y2="53.975" width="0.254" layer="16"/>
-<wire x1="33.655" y1="53.975" x2="36.195" y2="56.515" width="0.254" layer="16"/>
-<wire x1="36.195" y1="56.515" x2="50.8" y2="56.515" width="0.254" layer="16"/>
-<wire x1="50.8" y1="56.515" x2="51.435" y2="57.15" width="0.254" layer="16"/>
-<wire x1="51.435" y1="57.15" x2="51.435" y2="69.215" width="0.254" layer="16"/>
-<wire x1="51.435" y1="69.215" x2="52.705" y2="70.485" width="0.254" layer="16"/>
-<wire x1="52.705" y1="70.485" x2="54.6" y2="70.485" width="0.254" layer="16"/>
-<wire x1="54.6" y1="70.485" x2="54.695" y2="70.58" width="0.254" layer="16"/>
 </signal>
 <signal name="5V">
@@
 <signal name="B_TX">
 <contactref element="U1" pad="1"/>
-<contactref element="IC1" pad="14"/>
 <wire x1="57.15" y1="41.91" x2="50.8" y2="41.91" width="0.254" layer="1"/>
 <wire x1="50.8" y1="41.91" x2="49.53" y2="43.18" width="0.254" layer="1"/>
@@
 <via x="43.18" y="69.85" extent="1-16" drill="0.6"/>
 <wire x1="43.18" y1="69.85" x2="40.8624" y2="69.85" width="0.254" layer="1"/>
-<wire x1="40.8624" y1="69.85" x2="40.7924" y2="69.92" width="0.254" layer="1"/>
-</signal>
-<signal name="B_RX">
-<contactref element="U1" pad="2"/>
-<contactref element="IC1" pad="15"/>
-<contactref element="ISP1" pad="4"/>
-<wire x1="57.15" y1="43.41" x2="51.205" y2="43.41" width="0.254" layer="1"/>
-<wire x1="51.205" y1="43.41" x2="50.8" y2="43.815" width="0.254" layer="1"/>
-<wire x1="50.8" y1="43.815" x2="50.8" y2="49.53" width="0.254" layer="1"/>
-<wire x1="50.8" y1="49.53" x2="50.8" y2="57.15" width="0.254" layer="1"/>
-<wire x1="50.8" y1="57.15" x2="49.53" y2="58.42" width="0.254" layer="1"/>
-<via x="49.53" y="58.42" extent="1-16" drill="0.6"/>
-<wire x1="49.53" y1="58.42" x2="44.45" y2="63.5" width="0.254" layer="16"/>
-<wire x1="44.45" y1="63.5" x2="44.45" y2="64.77" width="0.254" layer="16"/>
-<via x="44.45" y="64.77" extent="1-16" drill="0.6"/>
-<wire x1="44.45" y1="64.77" x2="41.275" y2="64.77" width="0.254" layer="1"/>
-<wire x1="41.275" y1="64.77" x2="39.37" y2="66.675" width="0.254" layer="1"/>
-<wire x1="39.37" y1="66.675" x2="39.37" y2="68.58" width="0.254" layer="1"/>
-<wire x1="39.37" y1="68.58" x2="40.005" y2="69.215" width="0.254" layer="1"/>
-<wire x1="40.005" y1="69.215" x2="40.6974" y2="69.215" width="0.254" layer="1"/>
-<wire x1="40.6974" y1="69.215" x2="40.7924" y2="69.12" width="0.254" layer="1"/>
-<wire x1="15.24" y1="51.435" x2="15.24" y2="50.165" width="0.254" layer="16"/>
-<wire x1="15.24" y1="50.165" x2="18.415" y2="46.99" width="0.254" layer="16"/>
-<wire x1="18.415" y1="46.99" x2="31.75" y2="46.99" width="0.254" layer="16"/>
-<wire x1="31.75" y1="46.99" x2="33.655" y2="48.895" width="0.254" layer="16"/>
-<via x="33.655" y="48.895" extent="1-16" drill="0.6"/>
-<wire x1="33.655" y1="48.895" x2="36.83" y2="48.895" width="0.254" layer="1"/>
-<via x="36.83" y="48.895" extent="1-16" drill="0.6"/>
-<wire x1="36.83" y1="48.895" x2="53.975" y2="48.895" width="0.254" layer="16"/>
-<via x="53.975" y="48.895" extent="1-16" drill="0.6"/>
-<wire x1="53.975" y1="48.895" x2="51.435" y2="48.895" width="0.254" layer="1"/>
-<wire x1="51.435" y1="48.895" x2="50.8" y2="49.53" width="0.254" layer="1"/>
 </signal>
 <signal name="KEY">
@@
 <contactref element="IC2" pad="3"/>
 <contactref element="R16" pad="2"/>
+<contactref element="IC1" pad="27"/>
 <wire x1="0.635" y1="-170.0784" x2="-20.74" y2="-191.77" width="0" layer="19" extent="1-1"/>
+<wire x1="49.3776" y1="69.92" x2="0.635" y2="-170.0784" width="0" layer="19" extent="1-1"/>
 </signal>
 <signal name="SCL">
 <contactref element="IC2" pad="6"/>
 <contactref element="R17" pad="2"/>
+<contactref element="IC1" pad="28"/>
 <wire x1="4.445" y1="-170.0784" x2="-15.025" y2="-191.77" width="0" layer="19" extent="1-1"/>
+<wire x1="49.3776" y1="70.72" x2="4.445" y2="-170.0784" width="0" layer="19" extent="1-1"/>
 </signal>
 <signal name="N$1">
@@
 <wire x1="3.175" y1="-170.0784" x2="-9.31" y2="-191.77" width="0" layer="19" extent="1-1"/>
 </signal>
-<signal name="N$7">
-<contactref element="IC1" pad="19"/>
-</signal>
-<signal name="N$22">
-<contactref element="IC1" pad="22"/>
-</signal>
 <signal name="BT_TX">
 <contactref element="IC1" pad="32"/>
@@
 <contactref element="IC1" pad="12"/>
 </signal>
+<signal name="D12/MISO">
+<contactref element="IC1" pad="16"/>
+<contactref element="J6" pad="1"/>
+<contactref element="ISP1" pad="1"/>
+<wire x1="47.9425" y1="68.2625" x2="47.9425" y2="70.1675" width="0.254" layer="1"/>
+<wire x1="47.9425" y1="70.1675" x2="47.625" y2="70.485" width="0.254" layer="1"/>
+<wire x1="47.625" y1="70.485" x2="45.72" y2="70.485" width="0.254" layer="1"/>
+<wire x1="45.72" y1="70.485" x2="45.085" y2="69.85" width="0.254" layer="1"/>
+<wire x1="45.085" y1="69.85" x2="45.085" y2="69.215" width="0.254" layer="1"/>
+<wire x1="45.085" y1="69.215" x2="44.1325" y2="68.2625" width="0.254" layer="1"/>
+<wire x1="44.1325" y1="68.2625" x2="40.8499" y2="68.2625" width="0.254" layer="1"/>
+<wire x1="47.9425" y1="68.2625" x2="48.895" y2="67.31" width="0.254" layer="1"/>
+<wire x1="48.895" y1="67.31" x2="51.435" y2="67.31" width="0.254" layer="1"/>
+<wire x1="51.435" y1="67.31" x2="51.435" y2="69.215" width="0.254" layer="1"/>
+<wire x1="51.435" y1="69.215" x2="52.705" y2="70.485" width="0.254" layer="1"/>
+<wire x1="52.705" y1="70.485" x2="54.6" y2="70.485" width="0.254" layer="1"/>
+<wire x1="54.6" y1="70.485" x2="54.695" y2="70.58" width="0.254" layer="1"/>
+<wire x1="17.78" y1="53.975" x2="33.655" y2="53.975" width="0.254" layer="16"/>
+<wire x1="33.655" y1="53.975" x2="36.195" y2="56.515" width="0.254" layer="16"/>
+<wire x1="36.195" y1="56.515" x2="50.8" y2="56.515" width="0.254" layer="16"/>
+<wire x1="50.8" y1="56.515" x2="51.435" y2="57.15" width="0.254" layer="16"/>
+<wire x1="51.435" y1="57.15" x2="51.435" y2="69.215" width="0.254" layer="16"/>
+<wire x1="51.435" y1="69.215" x2="52.705" y2="70.485" width="0.254" layer="16"/>
+<wire x1="52.705" y1="70.485" x2="54.6" y2="70.485" width="0.254" layer="16"/>
+<wire x1="54.6" y1="70.485" x2="54.695" y2="70.58" width="0.254" layer="16"/>
+<wire x1="40.8499" y1="68.2625" x2="40.7924" y2="68.32" width="0" layer="19" extent="1-1"/>
+</signal>
+<signal name="D11/MOSI">
+<contactref element="IC1" pad="15"/>
+<contactref element="U1" pad="2"/>
+<contactref element="ISP1" pad="4"/>
+<wire x1="57.15" y1="43.41" x2="51.205" y2="43.41" width="0.254" layer="1"/>
+<wire x1="51.205" y1="43.41" x2="50.8" y2="43.815" width="0.254" layer="1"/>
+<wire x1="50.8" y1="43.815" x2="50.8" y2="49.53" width="0.254" layer="1"/>
+<wire x1="50.8" y1="49.53" x2="50.8" y2="57.15" width="0.254" layer="1"/>
+<wire x1="50.8" y1="57.15" x2="49.53" y2="58.42" width="0.254" layer="1"/>
+<via x="49.53" y="58.42" extent="1-16" drill="0.6"/>
+<wire x1="49.53" y1="58.42" x2="44.45" y2="63.5" width="0.254" layer="16"/>
+<wire x1="44.45" y1="63.5" x2="44.45" y2="64.77" width="0.254" layer="16"/>
+<via x="44.45" y="64.77" extent="1-16" drill="0.6"/>
+<wire x1="44.45" y1="64.77" x2="41.275" y2="64.77" width="0.254" layer="1"/>
+<wire x1="41.275" y1="64.77" x2="39.37" y2="66.675" width="0.254" layer="1"/>
+<wire x1="39.37" y1="66.675" x2="39.37" y2="68.58" width="0.254" layer="1"/>
+<wire x1="39.37" y1="68.58" x2="40.005" y2="69.215" width="0.254" layer="1"/>
+<wire x1="40.005" y1="69.215" x2="40.6974" y2="69.215" width="0.254" layer="1"/>
+<wire x1="15.24" y1="51.435" x2="15.24" y2="50.165" width="0.254" layer="16"/>
+<wire x1="15.24" y1="50.165" x2="18.415" y2="46.99" width="0.254" layer="16"/>
+<wire x1="18.415" y1="46.99" x2="31.75" y2="46.99" width="0.254" layer="16"/>
+<wire x1="31.75" y1="46.99" x2="33.655" y2="48.895" width="0.254" layer="16"/>
+<via x="33.655" y="48.895" extent="1-16" drill="0.6"/>
+<wire x1="33.655" y1="48.895" x2="36.83" y2="48.895" width="0.254" layer="1"/>
+<via x="36.83" y="48.895" extent="1-16" drill="0.6"/>
+<wire x1="36.83" y1="48.895" x2="53.975" y2="48.895" width="0.254" layer="16"/>
+<via x="53.975" y="48.895" extent="1-16" drill="0.6"/>
+<wire x1="53.975" y1="48.895" x2="51.435" y2="48.895" width="0.254" layer="1"/>
+<wire x1="51.435" y1="48.895" x2="50.8" y2="49.53" width="0.254" layer="1"/>
+<wire x1="40.6974" y1="69.215" x2="40.7924" y2="69.12" width="0" layer="19" extent="1-1"/>
+</signal>
+<signal name="D10">
+<contactref element="IC1" pad="14"/>
+</signal>
 </signals>

Commit message: Improving schematic
Parts:
- added FRAME1: FRAME-LETTERNO_PACKAGE, SparkFun-Aesthetics:DUMMY
- J6: value EXTRA-D12 -> EXTRA-D10
Connections:
- removed net B_TX: U1.1
- removed net D11/MOSI: IC1.15, ISP1.4, U1.2
- removed net D12/MISO: IC1.16, ISP1.1, J6.1
- removed net D2: J1.1
- removed net D3: J3.1
- removed net D4: IC1.2, J5.1
- removed net D5: IC1.9, J2.1
- removed net D6: IC1.10, J4.1
- net BT_RX: now also ISP1.4, U1.2
- net BT_TX: now also U1.1
- net D10: now also IC1.16, ISP1.1, J6.1
- net D7: now also IC1.9, J2.1, J3.1
- net D8: now also IC1.10, IC1.2, J1.1, J4.1, J5.1
Routing:
- net D11/MOSI: track 85.0 -> 0.00 mm, vias 5 -> 0
- net BT_RX: track 0.00 -> 85.0 mm, vias 0 -> 5
- net D12/MISO: track 70.9 -> 0.00 mm
- net D10: track 0.00 -> 70.9 mm
- net D8: track 0.00 -> 69.0 mm
- net B_TX: track 39.8 -> 0.00 mm, vias 2 -> 0
- net BT_TX: track 0.00 -> 39.8 mm, vias 0 -> 2
- net D7: track 0.00 -> 35.7 mm
- net D6: track 34.3 -> 0.00 mm
- net D5: track 23.1 -> 0.00 mm
- net D4: track 21.9 -> 0.00 mm
- net D2: track 12.8 -> 0.00 mm
- net D3: track 12.6 -> 0.00 mm

Commit message: Changing schematic
Parts:
- removed C1, C3: 100n, SparkFun-Passives:0805
- removed C2, C5: 0.1u, SparkFun-Passives:0603-CAP
- removed C4: 0.1u, SparkFun-Passives:0805
- removed C6: 10u, rcl:SMC_P
- removed D2: GREEN, SparkFun-LED:LED-0603
- removed IC1: MEGA8-AI, atmel:TQFP32-08
- removed R2: 10k, SparkFun-Passives:0805
- removed R3: 1k, SparkFun-Passives:0805
- removed S1: SWITCH-MOMENTARY-2PTH, SparkFun-Electromechanical:TACTILE-PTH
- removed Y1: 16MHZ, SparkFun-FreqCtrl:RESONATOR-SMD
- added C16, C7: 100n, SparkFun-Passives:0805
- added C17: 0.1u, SparkFun-Passives:0805
- added C18, C19: 0.1u, SparkFun-Passives:0603-CAP
- added C20: 10u, rcl:SMC_P
- added D3: GREEN, SparkFun-LED:LED-0603
- added FRAME2: FRAME-LETTERNO_PACKAGE, SparkFun-Aesthetics:DUMMY
- added R1: 10k, SparkFun-Passives:0805
- added R18: 1k, SparkFun-Passives:0805
- added S2: SWITCH-MOMENTARY-2PTH, SparkFun-Electromechanical:TACTILE-PTH
- added U2: MIC5219 3.3V, SparkFun-PowerIC:SOT23-5
- added Y2: 16MHZ, SparkFun-FreqCtrl:RESONATOR-SMD
- U3: value MIC5219 3.3V -> ATMEGA328P_TQFP; device SparkFun-PowerIC:SOT23-5 -> SparkFun-DigitalIC:TQFP32-08
- moved U3 47.5 mm to (-32.4, -229.9)
Connections:
- removed net KEY: IC1.13
- removed net N$6: D2.A, R3.1
- new net 11/MOSI: ISP1.4, U3.15
- new net 12/MISO: ISP1.1, U3.16
- new net D4: U3.2
- new net D5: U3.9
- new net D6: U3.10
- new net N$24: D3.A, R18.1
- net 3.3V: now also C19.1, C20.+, U2.5; no longer C5.1, C6.+, U3.5
- net 5V: now also C17.2, C18.2, R1.2, U2.1, U2.3, U3.18, U3.4, U3.6; no longer C2.2, C4.2, IC1.18, IC1.4, IC1.6, R2.2, U3.1, U3.3
- net A0: now also U3.23; no longer IC1.23
- net BT_RX: now also U3.1; no longer IC1.1, ISP1.4
- net BT_TX: now also U3.32; no longer IC1.32
- net D10: now also U3.14; no longer IC1.14, IC1.16, ISP1.1
- net D13/SCK: now also R18.2, U3.17; no longer IC1.17, R3.2
- net D7: now also U3.11; no longer IC1.11, IC1.9
- net D8: now also U3.12; no longer IC1.10, IC1.12, IC1.2
- net DTR: now also C7.1; no longer C1.1
- net GND: now also C16.1, C17.1, C18.1, C19.2, C20.-, D3.C, S2.1, U2.2, U3.21, U3.3, U3.5, Y2.2; no longer C2.1, C3.1, C4.1, C5.2, C6.-, D2.C, IC1.21, IC1.3, IC1.5, S1.1, U3.2, Y1.2
- net N$2: now also U3.7, Y2.1; no longer C3.2, IC1.20
- net N$3: now also U3.8, Y2.3; no longer IC1.7, Y1.1
- net N$4: now also C16.2, U3.20; no longer IC1.8, Y1.3
- net RESET: now also C7.2, R1.1, S2.3, U3.29; no longer C1.2, IC1.29, R2.1, S1.3
- net RX: now also U3.30; no longer IC1.30
- net SCL: now also U3.28; no longer IC1.28
- net SDA: now also U3.27; no longer IC1.27
- net TX: now also U3.31; no longer IC1.31
Routing:
- net RESET: track 28.4 -> 4.28 mm, vias 1 -> 0
- net N$2: track 18.0 -> 0.00 mm, vias 2 -> 0
- net D10: track 70.9 -> 55.0 mm
- net 5V: track 226.9 -> 221.2 mm
- net GND: track 27.8 -> 22.5 mm
- net N$4: track 4.10 -> 0.00 mm
- net DTR: track 7.13 -> 3.58 mm
- net N$6: track 2.03 -> 0.00 mm
- net N$3: track 1.95 -> 0.00 mm
- net D13/SCK: track 21.3 -> 19.6 mm
- net BT_RX: track 85.0 -> 83.7 mm
- net TX: track 52.8 -> 51.9 mm
- net RX: track 55.1 -> 54.4 mm
