File: SLAMP.brd (EAGLE design)
At the start: 160 x 100 mm, 59 parts, among them IC2 AT42QT1070-SSU, J1 CARA1, J2 CARA4, J3 CARA2, J4 CARA5, J5 CARA3, J6 EXTRA-D10, J7 A0, Q1 2N7002PW, U1 HC_05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

Commit message: adding system for power management
Parts:
- added D2: PINK, SparkFun-LED:LED-1206
- added Q2: BC548, transistor-npn:TO92-EBC
- added Q3: IRF520, transistor-power:TO220BV
- added R19, R2, R3: 2k, SparkFun-Passives:0805
Connections:
- new net N$22: D2.C, Q3.D
- new net N$6: Q2.B, R2.2, R3.2
- new net N$7: Q2.C, Q3.G, R19.2
- new net VCC_POWERSUPPLY: R2.1
- new net VUSB: C8.1, D2.A, F2.2
- net 5V: now also Q3.S, R19.1; no longer C8.1, F2.2
- net GND: now also Q2.E, R3.1
Routing:
- net 5V: track 221.2 -> 189.0 mm, vias 7 -> 5
- net VUSB: track 0.00 -> 30.9 mm, vias 0 -> 2
Changed lines of the file:
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@@
 <attribute name="PROD_ID" value="IC-09069" x="-32.385" y="-229.87" size="1.778" layer="27" display="off"/>
+</element>
+<element name="R2" library="SparkFun-Passives" package="0805" value="2k" x="-40.64" y="-234.95"/>
+<element name="R3" library="SparkFun-Passives" package="0805" value="2k" x="-43.815" y="-234.95"/>
+<element name="Q2" library="transistor-npn" package="TO92-EBC" value="BC548" x="-36.195" y="-242.57"/>
+<element name="Q3" library="transistor-power" package="TO220BV" value="IRF520" x="-34.925" y="-255.905"/>
+<element name="R19" library="SparkFun-Passives" package="0805" value="2k" x="-46.99" y="-263.525"/>
+<element name="D2" library="SparkFun-LED" package="LED-1206" value="PINK" x="-45.72" y="-268.605">
+<attribute name="PROD_ID" value="DIO-10415" x="-45.72" y="-268.605" size="1.778" layer="27" display="off"/>
 </element>
 </elements>
@@
 <contactref element="U3" pad="3"/>
 <contactref element="U3" pad="5"/>
+<contactref element="R3" pad="1"/>
+<contactref element="Q2" pad="E"/>
 <wire x1="-21.22" y1="-233.68" x2="-18.045" y2="-233.68" width="0" layer="19" extent="1-1"/>
 <wire x1="-28.0924" y1="-229.47" x2="-21.22" y2="-233.68" width="0" layer="19" extent="1-1"/>
 <wire x1="-36.6776" y1="-228.67" x2="-28.0924" y2="-229.47" width="0" layer="19" extent="1-1"/>
 <wire x1="-36.6776" y1="-230.27" x2="-36.6776" y2="-228.67" width="0" layer="19" extent="1-1"/>
+<wire x1="-44.715" y1="-234.95" x2="-36.6776" y2="-230.27" width="0" layer="19" extent="1-1"/>
 <wire x1="-7.62" y1="-232.168" x2="-18.045" y2="-233.68" width="0" layer="19" extent="1-1"/>
 <wire x1="-4.025" y1="-233.045" x2="-7.62" y2="-232.168" width="0" layer="19" extent="1-1"/>
@@
 <wire x1="-0.965" y1="-220.98" x2="-10.16" y2="-222.9151" width="0" layer="19" extent="1-1"/>
 <wire x1="3.81" y1="-221.361" x2="-0.965" y2="-220.98" width="0" layer="19" extent="1-1"/>
+<wire x1="-33.655" y1="-243.84" x2="-36.6776" y2="-230.27" width="0" layer="19" extent="1-1"/>
 <wire x1="-15.3162" y1="-204.1144" x2="-10.16" y2="-222.9151" width="0" layer="19" extent="1-1"/>
 <wire x1="-15.025" y1="-188.595" x2="-15.3162" y2="-204.1144" width="0" layer="19" extent="1-1"/>
@@
 </signal>
 <signal name="5V">
-<contactref element="F2" pad="2"/>
-<contactref element="C8" pad="1"/>
 <contactref element="U4" pad="15"/>
 <contactref element="C14" pad="1"/>
@@
 <wire x1="34.925" y1="45.085" x2="33.655" y2="43.815" width="0.8128" layer="16"/>
 <wire x1="33.655" y1="43.815" x2="16.51" y2="43.815" width="0.8128" layer="16"/>
-<wire x1="18.545" y1="66.04" x2="18.545" y2="65.91" width="0.254" layer="1"/>
 <wire x1="18.545" y1="65.91" x2="20.32" y2="64.135" width="0.254" layer="1"/>
 <wire x1="20.32" y1="64.135" x2="20.32" y2="60.325" width="0.254" layer="1"/>
@@
 <wire x1="24.4475" y1="69.7103" x2="24.4475" y2="68.2625" width="0.254" layer="1"/>
 <wire x1="24.4475" y1="68.2625" x2="24.13" y2="67.945" width="0.254" layer="1"/>
-<wire x1="31.7801" y1="68.6101" x2="32.385" y2="69.215" width="0.254" layer="1"/>
-<wire x1="32.385" y1="69.215" x2="34.925" y2="69.215" width="0.254" layer="1"/>
-<wire x1="34.925" y1="69.215" x2="35.56" y2="69.85" width="0.254" layer="1"/>
-<wire x1="35.56" y1="69.85" x2="35.56" y2="70.27" width="0.254" layer="1"/>
-<wire x1="35.56" y1="70.27" x2="35.775" y2="70.485" width="0.254" layer="1"/>
 <wire x1="24.13" y1="67.945" x2="23.495" y2="67.945" width="0.254" layer="1"/>
 <via x="23.495" y="67.945" extent="1-16" drill="0.6"/>
@@
 <wire x1="20.32" y1="66.675" x2="19.685" y2="66.04" width="0.254" layer="16"/>
 <via x="19.685" y="66.04" extent="1-16" drill="0.6"/>
-<wire x1="19.685" y1="66.04" x2="18.545" y2="66.04" width="0.254" layer="1"/>
-<wire x1="35.56" y1="69.85" x2="36.83" y2="69.85" width="0.254" layer="1"/>
-<wire x1="36.83" y1="69.85" x2="38.735" y2="67.945" width="0.254" layer="1"/>
-<wire x1="38.735" y1="67.945" x2="38.735" y2="65.405" width="0.254" layer="1"/>
-<wire x1="38.735" y1="65.405" x2="39.37" y2="64.77" width="0.254" layer="1"/>
-<wire x1="39.37" y1="64.77" x2="40.005" y2="64.77" width="0.254" layer="1"/>
-<wire x1="40.005" y1="64.77" x2="40.64" y2="64.135" width="0.254" layer="1"/>
-<wire x1="40.64" y1="64.135" x2="43.18" y2="64.135" width="0.254" layer="1"/>
-<wire x1="43.18" y1="64.135" x2="43.815" y2="63.5" width="0.254" layer="1"/>
-<wire x1="43.815" y1="63.5" x2="47.36" y2="63.5" width="0.254" layer="1"/>
-<wire x1="43.085" y1="65.945" x2="42.545" y2="65.405" width="0.254" layer="1"/>
-<wire x1="42.545" y1="65.405" x2="41.91" y2="65.405" width="0.254" layer="1"/>
-<wire x1="41.91" y1="65.405" x2="40.64" y2="66.675" width="0.254" layer="1"/>
-<via x="40.64" y="66.675" extent="1-16" drill="0.6"/>
-<wire x1="40.64" y1="66.675" x2="40.64" y2="67.31" width="0.254" layer="16"/>
-<wire x1="40.64" y1="67.31" x2="37.465" y2="70.485" width="0.254" layer="16"/>
-<via x="37.465" y="70.485" extent="1-16" drill="0.6"/>
-<wire x1="37.465" y1="70.485" x2="35.775" y2="70.485" width="0.254" layer="1"/>
 <wire x1="44.45" y1="76.835" x2="45.085" y2="76.835" width="0.254" layer="1"/>
 <wire x1="45.085" y1="76.835" x2="45.4025" y2="76.5175" width="0.254" layer="1"/>
@@
 <contactref element="U3" pad="4"/>
 <contactref element="U3" pad="18"/>
+<contactref element="R19" pad="1"/>
+<contactref element="Q3" pad="S"/>
 <wire x1="-13.07" y1="-233.68" x2="-16.245" y2="-233.68" width="0" layer="19" extent="1-1"/>
 <wire x1="-2.325" y1="-233.045" x2="-13.07" y2="-233.68" width="0" layer="19" extent="1-1"/>
@@
 <wire x1="-36.6776" y1="-231.07" x2="-28.0924" y2="-231.87" width="0" layer="19" extent="1-1"/>
 <wire x1="-36.6776" y1="-229.47" x2="-36.6776" y2="-231.07" width="0" layer="19" extent="1-1"/>
+<wire x1="-32.385" y1="-258.445" x2="-28.0924" y2="-231.87" width="0" layer="19" extent="1-1"/>
+<wire x1="-47.89" y1="-263.525" x2="-32.385" y2="-258.445" width="0" layer="19" extent="1-1"/>
 <wire x1="16.51" y1="43.815" x2="-9.21" y2="-222.9151" width="0" layer="19" extent="1-16"/>
 <wire x1="16.14" y1="48.525" x2="16.51" y2="46.62" width="0" layer="19" extent="1-1"/>
 <wire x1="16.295" y1="80.01" x2="15.875" y2="85.81" width="0" layer="19" extent="1-1"/>
-<wire x1="47.36" y1="63.5" x2="52.705" y2="67.31" width="0" layer="19" extent="1-16"/>
-<wire x1="24.4475" y1="68.2625" x2="31.7801" y2="68.6101" width="0" layer="19" extent="1-1"/>
+<wire x1="21.59" y1="59.055" x2="17.78" y2="51.435" width="0" layer="19" extent="1-1"/>
+<wire x1="19.685" y1="66.04" x2="18.545" y2="65.91" width="0" layer="19" extent="1-16"/>
 </signal>
 <signal name="VCCIO">
@@
 <contactref element="U3" pad="2"/>
 </signal>
+<signal name="VUSB">
+<contactref element="F2" pad="2"/>
+<contactref element="C8" pad="1"/>
+<wire x1="31.7801" y1="68.6101" x2="32.385" y2="69.215" width="0.254" layer="1"/>
+<wire x1="32.385" y1="69.215" x2="34.925" y2="69.215" width="0.254" layer="1"/>
+<wire x1="34.925" y1="69.215" x2="35.56" y2="69.85" width="0.254" layer="1"/>
+<wire x1="35.56" y1="69.85" x2="35.56" y2="70.27" width="0.254" layer="1"/>
+<wire x1="35.56" y1="70.27" x2="35.775" y2="70.485" width="0.254" layer="1"/>
+<wire x1="35.56" y1="69.85" x2="36.83" y2="69.85" width="0.254" layer="1"/>
+<wire x1="36.83" y1="69.85" x2="38.735" y2="67.945" width="0.254" layer="1"/>
+<wire x1="38.735" y1="67.945" x2="38.735" y2="65.405" width="0.254" layer="1"/>
+<wire x1="38.735" y1="65.405" x2="39.37" y2="64.77" width="0.254" layer="1"/>
+<wire x1="39.37" y1="64.77" x2="40.005" y2="64.77" width="0.254" layer="1"/>
+<wire x1="40.005" y1="64.77" x2="40.64" y2="64.135" width="0.254" layer="1"/>
+<wire x1="40.64" y1="64.135" x2="43.18" y2="64.135" width="0.254" layer="1"/>
+<wire x1="43.18" y1="64.135" x2="43.815" y2="63.5" width="0.254" layer="1"/>
+<wire x1="43.815" y1="63.5" x2="47.36" y2="63.5" width="0.254" layer="1"/>
+<wire x1="43.085" y1="65.945" x2="42.545" y2="65.405" width="0.254" layer="1"/>
+<wire x1="42.545" y1="65.405" x2="41.91" y2="65.405" width="0.254" layer="1"/>
+<wire x1="41.91" y1="65.405" x2="40.64" y2="66.675" width="0.254" layer="1"/>
+<via x="40.64" y="66.675" extent="1-16" drill="0.6"/>
+<wire x1="40.64" y1="66.675" x2="40.64" y2="67.31" width="0.254" layer="16"/>
+<wire x1="40.64" y1="67.31" x2="37.465" y2="70.485" width="0.254" layer="16"/>
+<via x="37.465" y="70.485" extent="1-16" drill="0.6"/>
+<wire x1="37.465" y1="70.485" x2="35.775" y2="70.485" width="0.254" layer="1"/>
+<contactref element="D2" pad="A"/>
+<wire x1="18.545" y1="66.04" x2="31.7801" y2="68.6101" width="0" layer="19" extent="1-1"/>
+<wire x1="-47.22" y1="-268.605" x2="18.545" y2="66.04" width="0" layer="19" extent="1-1"/>
+</signal>
+<signal name="N$6">
+<contactref element="R2" pad="2"/>
+<contactref element="Q2" pad="B"/>
+<contactref element="R3" pad="2"/>
+<wire x1="-39.74" y1="-234.95" x2="-36.195" y2="-243.84" width="0" layer="19" extent="1-1"/>
+<wire x1="-42.915" y1="-234.95" x2="-39.74" y2="-234.95" width="0" layer="19" extent="1-1"/>
+</signal>
+<signal name="N$7">
+<contactref element="Q2" pad="C"/>
+<contactref element="R19" pad="2"/>
+<contactref element="Q3" pad="G"/>
+<wire x1="-37.465" y1="-258.445" x2="-46.09" y2="-263.525" width="0" layer="19" extent="1-1"/>
+<wire x1="-38.735" y1="-243.84" x2="-37.465" y2="-258.445" width="0" layer="19" extent="1-1"/>
+</signal>
+<signal name="N$22">
+<contactref element="Q3" pad="D"/>
+<contactref element="D2" pad="C"/>
+<wire x1="-34.925" y1="-258.445" x2="-44.22" y2="-268.605" width="0" layer="19" extent="1-1"/>
+</signal>
+<signal name="VCC_POWERSUPPLY">
+<contactref element="R2" pad="1"/>
+</signal>
 </signals>

Commit message: Working on the power management
Parts:
- removed C8: 10n, SparkFun-Passives:0603-CAP
- removed D2: PINK, SparkFun-LED:LED-1206
- removed F2: 500mA, SparkFun-PowerIC:PTC-1206
- removed Q2: BC548, transistor-npn:TO92-EBC
- removed Q3: IRF520, transistor-power:TO220BV
- removed R19, R2, R3: 2k, SparkFun-Passives:0805
Connections:
- removed net N$18: F2.1, JP1.4
- removed net N$22: D2.C, Q3.D
- removed net N$6: Q2.B, R2.2, R3.2
- removed net N$7: Q2.C, Q3.G, R19.2
- removed net VCC_POWERSUPPLY: R2.1
- removed net VUSB: C8.1, D2.A, F2.2
- net 5V: no longer Q3.S, R19.1
- net GND: no longer C8.2, Q2.E, R3.1
Routing:
- net VUSB: track 30.9 -> 0.00 mm, vias 2 -> 0
- net N$18: track 4.47 -> 0.00 mm
Changed lines of the file:
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@@
 <element name="C13" library="SparkFun-Passives" package="0603-CAP" value="47p" x="17.145" y="76.835"/>
 <element name="C14" library="SparkFun-Passives" package="0603-CAP" value="100n" x="17.145" y="80.01"/>
-<element name="C8" library="SparkFun-Passives" package="0603-CAP" value="10n" x="34.925" y="70.485" rot="R180"/>
 <element name="C9" library="SparkFun-Passives" package="0603-CAP" value="100n" x="34.925" y="67.945" rot="R180"/>
 <element name="D1" library="SparkFun-LED" package="LED-0603" value="BLUE" x="38.735" y="57.15" rot="R270">
 <attribute name="PROD_ID" value="DIO-08575" x="38.735" y="57.15" size="1.778" layer="27" rot="R270" display="off"/>
-</element>
-<element name="F2" library="SparkFun-PowerIC" package="PTC-1206" value="500mA" x="17.145" y="66.04">
-<attribute name="PROD_ID" value="RES-11150" x="17.145" y="66.04" size="1.778" layer="27" display="off"/>
 </element>
 <element name="ISP1" library="adafruit" package="AVRISP" value="AVRISP-6" x="15.24" y="52.705" rot="R270"/>
@@
 <attribute name="PROD_ID" value="IC-09069" x="-32.385" y="-229.87" size="1.778" layer="27" display="off"/>
 </element>
-<element name="R2" library="SparkFun-Passives" package="0805" value="2k" x="-40.64" y="-234.95"/>
-<element name="R3" library="SparkFun-Passives" package="0805" value="2k" x="-43.815" y="-234.95"/>
-<element name="Q2" library="transistor-npn" package="TO92-EBC" value="BC548" x="-36.195" y="-242.57"/>
-<element name="Q3" library="transistor-power" package="TO220BV" value="IRF520" x="-34.925" y="-255.905"/>
-<element name="R19" library="SparkFun-Passives" package="0805" value="2k" x="-46.99" y="-263.525"/>
-<element name="D2" library="SparkFun-LED" package="LED-1206" value="PINK" x="-45.72" y="-268.605">
-<attribute name="PROD_ID" value="DIO-10415" x="-45.72" y="-268.605" size="1.778" layer="27" display="off"/>
-</element>
 </elements>
 <signals>
@@
 <contactref element="U4" pad="6"/>
 <contactref element="U4" pad="16"/>
-<contactref element="C8" pad="2"/>
 <contactref element="C12" pad="2"/>
 <contactref element="C13" pad="2"/>
@@
 <contactref element="U3" pad="3"/>
 <contactref element="U3" pad="5"/>
-<contactref element="R3" pad="1"/>
-<contactref element="Q2" pad="E"/>
 <wire x1="-21.22" y1="-233.68" x2="-18.045" y2="-233.68" width="0" layer="19" extent="1-1"/>
 <wire x1="-28.0924" y1="-229.47" x2="-21.22" y2="-233.68" width="0" layer="19" extent="1-1"/>
 <wire x1="-36.6776" y1="-228.67" x2="-28.0924" y2="-229.47" width="0" layer="19" extent="1-1"/>
 <wire x1="-36.6776" y1="-230.27" x2="-36.6776" y2="-228.67" width="0" layer="19" extent="1-1"/>
-<wire x1="-44.715" y1="-234.95" x2="-36.6776" y2="-230.27" width="0" layer="19" extent="1-1"/>
 <wire x1="-7.62" y1="-232.168" x2="-18.045" y2="-233.68" width="0" layer="19" extent="1-1"/>
 <wire x1="-4.025" y1="-233.045" x2="-7.62" y2="-232.168" width="0" layer="19" extent="1-1"/>
@@
 <wire x1="-0.965" y1="-220.98" x2="-10.16" y2="-222.9151" width="0" layer="19" extent="1-1"/>
 <wire x1="3.81" y1="-221.361" x2="-0.965" y2="-220.98" width="0" layer="19" extent="1-1"/>
-<wire x1="-33.655" y1="-243.84" x2="-36.6776" y2="-230.27" width="0" layer="19" extent="1-1"/>
 <wire x1="-15.3162" y1="-204.1144" x2="-10.16" y2="-222.9151" width="0" layer="19" extent="1-1"/>
 <wire x1="-15.025" y1="-188.595" x2="-15.3162" y2="-204.1144" width="0" layer="19" extent="1-1"/>
@@
 <wire x1="17.875" y1="85.81" x2="17.995" y2="80.01" width="0" layer="19" extent="1-1"/>
 <wire x1="27.4" y1="85.81" x2="25.4" y2="79.07" width="0" layer="19" extent="1-1"/>
-<wire x1="34.075" y1="70.485" x2="25.0825" y2="69.7103" width="0" layer="19" extent="1-1"/>
-<wire x1="34.075" y1="67.945" x2="34.075" y2="70.485" width="0" layer="19" extent="1-1"/>
+<wire x1="34.075" y1="67.945" x2="25.0825" y2="69.7103" width="0" layer="19" extent="1-1"/>
 <wire x1="36.925" y1="85.81" x2="27.4" y2="85.81" width="0" layer="19" extent="1-1"/>
 <wire x1="46.45" y1="85.81" x2="36.925" y2="85.81" width="0" layer="19" extent="1-1"/>
@@
 <contactref element="U3" pad="4"/>
 <contactref element="U3" pad="18"/>
-<contactref element="R19" pad="1"/>
-<contactref element="Q3" pad="S"/>
 <wire x1="-13.07" y1="-233.68" x2="-16.245" y2="-233.68" width="0" layer="19" extent="1-1"/>
 <wire x1="-2.325" y1="-233.045" x2="-13.07" y2="-233.68" width="0" layer="19" extent="1-1"/>
@@
 <wire x1="-36.6776" y1="-231.07" x2="-28.0924" y2="-231.87" width="0" layer="19" extent="1-1"/>
 <wire x1="-36.6776" y1="-229.47" x2="-36.6776" y2="-231.07" width="0" layer="19" extent="1-1"/>
-<wire x1="-32.385" y1="-258.445" x2="-28.0924" y2="-231.87" width="0" layer="19" extent="1-1"/>
-<wire x1="-47.89" y1="-263.525" x2="-32.385" y2="-258.445" width="0" layer="19" extent="1-1"/>
 <wire x1="16.51" y1="43.815" x2="-9.21" y2="-222.9151" width="0" layer="19" extent="1-16"/>
 <wire x1="16.14" y1="48.525" x2="16.51" y2="46.62" width="0" layer="19" extent="1-1"/>
@@
 <wire x1="15.24" y1="71.755" x2="16.295" y2="71.755" width="0.254" layer="1"/>
 <wire x1="16.295" y1="68.58" x2="16.295" y2="71.755" width="0.254" layer="1"/>
-</signal>
-<signal name="N$18">
-<contactref element="F2" pad="1"/>
-<contactref element="JP1" pad="4"/>
-<wire x1="12.065" y1="67.945" x2="12.7" y2="67.945" width="0.254" layer="1"/>
-<wire x1="12.7" y1="67.945" x2="14.605" y2="66.04" width="0.254" layer="1"/>
-<wire x1="14.605" y1="66.04" x2="15.745" y2="66.04" width="0.254" layer="1"/>
 </signal>
 <signal name="CBUS1">
@@
 <contactref element="U3" pad="2"/>
 </signal>
-<signal name="VUSB">
-<contactref element="F2" pad="2"/>
-<contactref element="C8" pad="1"/>
-<wire x1="31.7801" y1="68.6101" x2="32.385" y2="69.215" width="0.254" layer="1"/>
-<wire x1="32.385" y1="69.215" x2="34.925" y2="69.215" width="0.254" layer="1"/>
-<wire x1="34.925" y1="69.215" x2="35.56" y2="69.85" width="0.254" layer="1"/>
-<wire x1="35.56" y1="69.85" x2="35.56" y2="70.27" width="0.254" layer="1"/>
-<wire x1="35.56" y1="70.27" x2="35.775" y2="70.485" width="0.254" layer="1"/>
-<wire x1="35.56" y1="69.85" x2="36.83" y2="69.85" width="0.254" layer="1"/>
-<wire x1="36.83" y1="69.85" x2="38.735" y2="67.945" width="0.254" layer="1"/>
-<wire x1="38.735" y1="67.945" x2="38.735" y2="65.405" width="0.254" layer="1"/>
-<wire x1="38.735" y1="65.405" x2="39.37" y2="64.77" width="0.254" layer="1"/>
-<wire x1="39.37" y1="64.77" x2="40.005" y2="64.77" width="0.254" layer="1"/>
-<wire x1="40.005" y1="64.77" x2="40.64" y2="64.135" width="0.254" layer="1"/>
-<wire x1="40.64" y1="64.135" x2="43.18" y2="64.135" width="0.254" layer="1"/>
-<wire x1="43.18" y1="64.135" x2="43.815" y2="63.5" width="0.254" layer="1"/>
-<wire x1="43.815" y1="63.5" x2="47.36" y2="63.5" width="0.254" layer="1"/>
-<wire x1="43.085" y1="65.945" x2="42.545" y2="65.405" width="0.254" layer="1"/>
-<wire x1="42.545" y1="65.405" x2="41.91" y2="65.405" width="0.254" layer="1"/>
-<wire x1="41.91" y1="65.405" x2="40.64" y2="66.675" width="0.254" layer="1"/>
-<via x="40.64" y="66.675" extent="1-16" drill="0.6"/>
-<wire x1="40.64" y1="66.675" x2="40.64" y2="67.31" width="0.254" layer="16"/>
-<wire x1="40.64" y1="67.31" x2="37.465" y2="70.485" width="0.254" layer="16"/>
-<via x="37.465" y="70.485" extent="1-16" drill="0.6"/>
-<wire x1="37.465" y1="70.485" x2="35.775" y2="70.485" width="0.254" layer="1"/>
-<contactref element="D2" pad="A"/>
-<wire x1="18.545" y1="66.04" x2="31.7801" y2="68.6101" width="0" layer="19" extent="1-1"/>
-<wire x1="-47.22" y1="-268.605" x2="18.545" y2="66.04" width="0" layer="19" extent="1-1"/>
-</signal>
-<signal name="N$6">
-<contactref element="R2" pad="2"/>
-<contactref element="Q2" pad="B"/>
-<contactref element="R3" pad="2"/>
-<wire x1="-39.74" y1="-234.95" x2="-36.195" y2="-243.84" width="0" layer="19" extent="1-1"/>
-<wire x1="-42.915" y1="-234.95" x2="-39.74" y2="-234.95" width="0" layer="19" extent="1-1"/>
-</signal>
-<signal name="N$7">
-<contactref element="Q2" pad="C"/>
-<contactref element="R19" pad="2"/>
-<contactref element="Q3" pad="G"/>
-<wire x1="-37.465" y1="-258.445" x2="-46.09" y2="-263.525" width="0" layer="19" extent="1-1"/>
-<wire x1="-38.735" y1="-243.84" x2="-37.465" y2="-258.445" width="0" layer="19" extent="1-1"/>
-</signal>
-<signal name="N$22">
-<contactref element="Q3" pad="D"/>
-<contactref element="D2" pad="C"/>
-<wire x1="-34.925" y1="-258.445" x2="-44.22" y2="-268.605" width="0" layer="19" extent="1-1"/>
-</signal>
-<signal name="VCC_POWERSUPPLY">
-<contactref element="R2" pad="1"/>
-</signal>
 </signals>
